File: HydraFlasher_KiCAD.kicad_pcb (KiCad board)
At the start: 4 copper layers, 93 x 121 mm, 47 parts, among them J1 Conn_01x08_Socket, J2 Conn_01x08_Socket, J3 Conn_01x08_Socket, J4 Conn_01x08_Socket, J5 Conn_01x08_Socket, J6 Conn_01x08_Socket, J7 Conn_01x08_Socket, J8 Conn_01x08_Socket, U1 AP7361C-33E, U2 74AHCT1G125

Commit message: Polishing up
Parts:
- A1: footprint Rawr:Raspberry Pico SMD (with model) -> rawr:Raspberry Pico SMD (with model)
- C1, C2: value 10 µF -> 22 µF
- C10, C11, C4, C5, C6, C7, C8, C9: value 100NF -> 100nF
- C3: value 100 nF -> 100nF; footprint Capacitor_SMD:C_0805_2012Metric_Pad1.18x1.45mm_HandSolder -> Capacitor_SMD:C_0805_2012Metric
- J1, J2, J3, J4, J5, J6, J7, J8: footprint Rawr:DIP8-Hydra -> rawr:DIP8-Hydra
- U1: value AP7361C-33E -> AMS1117-3.3
- U2: footprint Package_TO_SOT_SMD:SOT-23-5 -> Package_TO_SOT_SMD:SOT-23-5_HandSoldering
- moved C1 3.08 mm to (79.7, 45.6), turned to -90 degrees
- moved C2 3.03 mm to (79.7, 52.1), turned to 90 degrees
- moved U1 0.61 mm to (74.8, 48.2), turned to -90 degrees
Connections:
- U1 pad 1: +VBUS -> GND
- U1 pad 2: GND -> +3V3_SOCK
- U1 pad 3: +3V3_SOCK -> +VBUS
Routing:
- net +VBUS: track 319.5 -> 323.9 mm
- net +3V3_SOCK: track 437.1 -> 441.5 mm
- net MOSI: track 317.0 -> 319.6 mm
- net SCK: track 302.9 -> 304.9 mm
- net GND: vias 1 -> 77
- added copper zone on B.Cu, net +3V3_SOCK
Other:
- outline, holes or cut-outs redrawn
- board text added: "JLCJLCJLCJLC"
- board text added: "Only for 3.3v chips!"
- board text added: "Rev1.2"
- board text removed: "Rev1.0"
