File: HydraFlasher_KiCAD.kicad_sch (KiCad schematic)
At the start: 23 parts, among them U1 74AHCT1G125, U2 AP7361C-33E

Commit message: Layout
Parts:
- renumbered C4 to C1, C7 to C2, C6 to C3, C1 to C4, C2 to C5, C3 to C6, C5 to C7, U2 to U1, U1 to U2
Other:
- note added: "HydraFlasher"
- title: Hydra Flasher Body (8 sockets) -> HydraFlasher body (8-sockets)

Commit message: Polishing up
Parts:
- removed U1: AP7361C-33E, Package_TO_SOT_SMD:SOT-223-3_TabPin2, symbol Regulator_Linear:AP7361C-33E
- added U1: AMS1117-3.3, Package_TO_SOT_SMD:SOT-223-3_TabPin2, symbol Regulator_Linear:AMS1117-3.3
- A1: footprint Rawr:Raspberry Pico SMD (with model) -> rawr:Raspberry Pico SMD (with model); LCSC (none) -> C7203002
- C1, C2: value 10 µF -> 22 µF; LCSC (none) -> C784585; LSCS (none) -> C784585; MPN (none) -> CC0805MKX5R8BB226
- C10, C11, C4, C5, C6, C7, C8, C9: value 100NF -> 100nF; LCSC (none) -> C49678
- C3: value 100 nF -> 100nF; footprint Capacitor_SMD:C_0805_2012Metric_Pad1.18x1.45mm_HandSolder -> Capacitor_SMD:C_0805_2012Metric; LCSC (none) -> C49678
- D1, D2, D3, D4, D5, D6, D7, D8: JLCPCB Rotation Offset (none) -> 180; LCSC (none) -> C2843785
- R1: LCSC (none) -> C17630
- U2: JLCPCB Rotation Offset (none) -> 180; LCSC (none) -> C7484; LSCS (none) -> C7484; MPN (none) -> SN74AHCT1G125DBVR
Connections:
- net +3V3_SOCK: now also U1.2 (VO)
- net +VBUS: now also U1.3 (VI)
- net GND: now also U1.1 (GND)
