File: socket.kicad_sch (KiCad schematic)
At the start: 3 parts, among them J1 Conn_01x08_Socket

Commit message: Polishing up
Parts:
- C12: LCSC (none) -> C1590
- J1: footprint Rawr:DIP8-Hydra -> rawr:DIP8-Hydra
- R2: LCSC (none) -> C17414
Changed lines of the file:
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@@
+			)
+		)
+		(property "LCSC" "C1590"
+			(at 161.798 114.808 0)
+			(effects
+				(font
+					(size 1.27 1.27)
+				)
+				(hide yes)
 			)
 		)
@@
 		(dnp no)
 		(fields_autoplaced yes)
-		(property "Reference" "#PWR014"
+		(property "Reference" "#PWR14"
 			(at 120.65 99.06 0)
 			(effects
@@
 			(project "HydraFlasher_KiCAD"
 				(path "/c22f8515-e30a-4928-96cd-86ae651c58e5/1f58108a-f2a0-49d6-a496-bab54aa8600f"
-					(reference "#PWR023")
+					(reference "#PWR23")
 					(unit 1)
 				)
 				(path "/c22f8515-e30a-4928-96cd-86ae651c58e5/2e155d08-bb5a-4122-ac1c-e075784ec07a"
-					(reference "#PWR035")
+					(reference "#PWR35")
 					(unit 1)
 				)
 				(path "/c22f8515-e30a-4928-96cd-86ae651c58e5/3ad5e6cb-7f8a-4a0d-aa87-3a8aeabe9d89"
-					(reference "#PWR026")
+					(reference "#PWR26")
 					(unit 1)
 				)
 				(path "/c22f8515-e30a-4928-96cd-86ae651c58e5/ae1cbe08-1fe9-4d78-a89b-85cbd406c476"
-					(reference "#PWR014")
+					(reference "#PWR14")
 					(unit 1)
 				)
 				(path "/c22f8515-e30a-4928-96cd-86ae651c58e5/ae5e4624-fcac-4dd9-9211-5ca85c98e0eb"
-					(reference "#PWR020")
+					(reference "#PWR20")
 					(unit 1)
 				)
 				(path "/c22f8515-e30a-4928-96cd-86ae651c58e5/c9262e07-ce5f-47d9-9eb2-43b6f4d75b76"
-					(reference "#PWR029")
+					(reference "#PWR29")
 					(unit 1)
 				)
 				(path "/c22f8515-e30a-4928-96cd-86ae651c58e5/d2a0ebb2-4fe0-4daa-88f7-b8aab7da5771"
-					(reference "#PWR032")
+					(reference "#PWR32")
 					(unit 1)
 				)
 				(path "/c22f8515-e30a-4928-96cd-86ae651c58e5/ed61606f-2c2f-4e28-a486-75a0b32162b0"
-					(reference "#PWR017")
+					(reference "#PWR17")
 					(unit 1)
 				)
@@
 		(on_board yes)
 		(dnp no)
-		(property "Reference" "#PWR015"
+		(property "Reference" "#PWR15"
 			(at 157.48 105.41 0)
 			(effects
@@
 			(project "HydraFlasher_KiCAD"
 				(path "/c22f8515-e30a-4928-96cd-86ae651c58e5/1f58108a-f2a0-49d6-a496-bab54aa8600f"
-					(reference "#PWR024")
+					(reference "#PWR24")
 					(unit 1)
 				)
 				(path "/c22f8515-e30a-4928-96cd-86ae651c58e5/2e155d08-bb5a-4122-ac1c-e075784ec07a"
-					(reference "#PWR036")
+					(reference "#PWR36")
 					(unit 1)
 				)
 				(path "/c22f8515-e30a-4928-96cd-86ae651c58e5/3ad5e6cb-7f8a-4a0d-aa87-3a8aeabe9d89"
-					(reference "#PWR027")
+					(reference "#PWR27")
 					(unit 1)
 				)
 				(path "/c22f8515-e30a-4928-96cd-86ae651c58e5/ae1cbe08-1fe9-4d78-a89b-85cbd406c476"
-					(reference "#PWR015")
+					(reference "#PWR15")
 					(unit 1)
 				)
 				(path "/c22f8515-e30a-4928-96cd-86ae651c58e5/ae5e4624-fcac-4dd9-9211-5ca85c98e0eb"
-					(reference "#PWR021")
+					(reference "#PWR21")
 					(unit 1)
 				)
 				(path "/c22f8515-e30a-4928-96cd-86ae651c58e5/c9262e07-ce5f-47d9-9eb2-43b6f4d75b76"
-					(reference "#PWR030")
+					(reference "#PWR30")
 					(unit 1)
 				)
 				(path "/c22f8515-e30a-4928-96cd-86ae651c58e5/d2a0ebb2-4fe0-4daa-88f7-b8aab7da5771"
-					(reference "#PWR033")
+					(reference "#PWR33")
 					(unit 1)
 				)
 				(path "/c22f8515-e30a-4928-96cd-86ae651c58e5/ed61606f-2c2f-4e28-a486-75a0b32162b0"
-					(reference "#PWR018")
+					(reference "#PWR18")
 					(unit 1)
 				)
@@
 			)
 		)
-		(property "Footprint" "Rawr:DIP8-Hydra"
+		(property "Footprint" "rawr:DIP8-Hydra"
 			(at 143.51 88.9 0)
 			(effects
@@
 			)
 		)
+		(property "LCSC" "C17414"
+			(at 150.114 109.982 0)
+			(effects
+				(font
+					(size 1.27 1.27)
+				)
+				(hide yes)
+			)
+		)
 		(pin "1"
 		)
@@
 		(dnp no)
 		(fields_autoplaced yes)
-		(property "Reference" "#PWR016"
+		(property "Reference" "#PWR16"
 			(at 158.75 121.92 0)
 			(effects
@@
 			(project "HydraFlasher_KiCAD"
 				(path "/c22f8515-e30a-4928-96cd-86ae651c58e5/1f58108a-f2a0-49d6-a496-bab54aa8600f"
-					(reference "#PWR025")
+					(reference "#PWR25")
 					(unit 1)
 				)
 				(path "/c22f8515-e30a-4928-96cd-86ae651c58e5/2e155d08-bb5a-4122-ac1c-e075784ec07a"
-					(reference "#PWR037")
+					(reference "#PWR37")
 					(unit 1)
 				)
 				(path "/c22f8515-e30a-4928-96cd-86ae651c58e5/3ad5e6cb-7f8a-4a0d-aa87-3a8aeabe9d89"
-					(reference "#PWR028")
+					(reference "#PWR28")
 					(unit 1)
 				)
 				(path "/c22f8515-e30a-4928-96cd-86ae651c58e5/ae1cbe08-1fe9-4d78-a89b-85cbd406c476"
-					(reference "#PWR016")
+					(reference "#PWR16")
 					(unit 1)
 				)
 				(path "/c22f8515-e30a-4928-96cd-86ae651c58e5/ae5e4624-fcac-4dd9-9211-5ca85c98e0eb"
-					(reference "#PWR022")
+					(reference "#PWR22")
 					(unit 1)
 				)
 				(path "/c22f8515-e30a-4928-96cd-86ae651c58e5/c9262e07-ce5f-47d9-9eb2-43b6f4d75b76"
-					(reference "#PWR031")
+					(reference "#PWR31")
 					(unit 1)
 				)
 				(path "/c22f8515-e30a-4928-96cd-86ae651c58e5/d2a0ebb2-4fe0-4daa-88f7-b8aab7da5771"
-					(reference "#PWR034")
+					(reference "#PWR34")
 					(unit 1)
 				)
 				(path "/c22f8515-e30a-4928-96cd-86ae651c58e5/ed61606f-2c2f-4e28-a486-75a0b32162b0"
-					(reference "#PWR019")
-					(unit 1)
-				)
+					(reference "#PWR19")
+					(unit 1)
+				)
